File: relay-board/relay-board.kicad_pcb (KiCad board)
At the start: 2 copper layers, 0 parts

Commit message: [relay-board] Updated schema, created PCB and added libraries with modules.
Parts:
- added C1: 10uF, CP, F.Cu at (222.2, 174.0)
- added D1: LED, LED-3MM-Large-pads, F.Cu at (100.3, 178.4)
- added D10: 1N4148, D3, F.Cu at (110.5, 161.3)
- added D11: 1N4148, D3, F.Cu at (127.0, 161.3)
- added D12: 1N4148, D3, F.Cu at (143.5, 161.3)
- added D13: 1N4148, D3, F.Cu at (160.0, 161.3)
- added D14: 1N4148, D3, F.Cu at (176.5, 161.3)
- added D15: 1N4148, D3, F.Cu at (193.0, 161.3)
- added D16: 1N4148, D3, F.Cu at (209.6, 161.3)
- added D2: LED, LED-3MM-Large-pads, F.Cu at (116.8, 178.4)
- added D3: LED, LED-3MM-Large-pads, F.Cu at (133.3, 178.4)
- added D4: LED, LED-3MM-Large-pads, F.Cu at (149.9, 178.4)
- added D5: LED, LED-3MM-Large-pads, F.Cu at (166.4, 178.4)
- added D6: LED, LED-3MM-Large-pads, F.Cu at (182.9, 178.4)
- added D7: LED, LED-3MM-Large-pads, F.Cu at (199.4, 178.4)
- added D8: LED, LED-3MM-Large-pads, F.Cu at (215.9, 178.4)
- added D9: 1N4148, D3, F.Cu at (94.0, 161.3)
- added IC1: OPTO-TRANSISTOR4, DIP-4__300_ELL, F.Cu at (100.3, 170.2)
- added IC2: OPTO-TRANSISTOR4, DIP-4__300_ELL, F.Cu at (116.8, 170.2)
- added IC3: OPTO-TRANSISTOR4, DIP-4__300_ELL, F.Cu at (133.3, 170.2)
- added IC4: OPTO-TRANSISTOR4, DIP-4__300_ELL, F.Cu at (149.9, 170.2)
- added IC5: OPTO-TRANSISTOR4, DIP-4__300_ELL, F.Cu at (166.4, 170.2)
- added IC6: OPTO-TRANSISTOR4, DIP-4__300_ELL, F.Cu at (182.9, 170.2)
- added IC7: OPTO-TRANSISTOR4, DIP-4__300_ELL, F.Cu at (199.4, 170.2)
- added IC8: OPTO-TRANSISTOR4, DIP-4__300_ELL, F.Cu at (215.9, 170.2)
- added K1: RELAY_JS5N-K, JS-K-Case, F.Cu at (104.1, 134.6)
- added K10: CONN_01X03, AK300-3, F.Cu at (114.3, 118.1)
- added K11: CONN_01X03, AK300-3, F.Cu at (130.8, 118.1)
- added K12: CONN_01X03, AK300-3, F.Cu at (147.3, 118.1)
- added K13: CONN_01X03, AK300-3, F.Cu at (163.8, 118.1)
- added K14: CONN_01X03, AK300-3, F.Cu at (180.3, 118.1)
- added K15: CONN_01X03, AK300-3, F.Cu at (196.8, 118.1)
- added K16: CONN_01X03, AK300-3, F.Cu at (213.4, 118.1)
- added K2: RELAY_JS5N-K, JS-K-Case, F.Cu at (120.7, 134.6)
- added K3: RELAY_JS5N-K, JS-K-Case, F.Cu at (137.2, 134.6)
- added K4: RELAY_JS5N-K, JS-K-Case, F.Cu at (153.7, 134.6)
- added K5: RELAY_JS5N-K, JS-K-Case, F.Cu at (170.2, 134.6)
- added K6: RELAY_JS5N-K, JS-K-Case, F.Cu at (186.7, 134.6)
- added K7: RELAY_JS5N-K, JS-K-Case, F.Cu at (203.2, 134.6)
- added K8: RELAY_JS5N-K, JS-K-Case, F.Cu at (219.7, 134.6)
- added K9: CONN_01X03, AK300-3, F.Cu at (97.8, 118.1)
- added P1: CONN_01X04, PINHEAD1-4-90, F.Cu at (208.3, 187.3)
- added P2: CONN_01X04, PINHEAD1-4-90, F.Cu at (220.3, 187.3)
- added P3: CONN_02X03, pin_array_3x2-large-pads, F.Cu at (130.8, 192.4)
- added P4: CONN_01X02, PINHEAD1-2-90, F.Cu at (221.6, 143.5)
- added P5: CONN_01X02, PINHEAD1-2-90, F.Cu at (221.6, 149.9)
- added P6: CONN_01X02, PINHEAD1-2-UP, F.Cu at (228.6, 143.5)
- added P7: CONN_01X02, PINHEAD1-2-UP, F.Cu at (228.6, 149.9)
- added Q1: BS107, TO92PN, F.Cu at (100.3, 158.8)
- added Q2: BS107, TO92PN, F.Cu at (116.8, 158.8)
- added Q3: BS107, TO92PN, F.Cu at (133.3, 158.8)
- added Q4: BS107, TO92PN, F.Cu at (149.9, 158.8)
- added Q5: BS107, TO92PN, F.Cu at (166.4, 158.8)
- added Q6: BS107, TO92PN, F.Cu at (182.9, 158.8)
- added Q7: BS107, TO92PN, F.Cu at (199.4, 158.8)
- added Q8: BS107, TO92PN, F.Cu at (215.9, 158.8)
- added R1: 10k, R3-LARGE_PADS, F.Cu at (138.4, 187.3)
- added R10: 1k, R3-LARGE_PADS, F.Cu at (199.4, 162.6)
- added R11: 1k, R3-LARGE_PADS, F.Cu at (215.9, 162.6)
- added R12: 100k, R3-LARGE_PADS, F.Cu at (106.7, 161.3)
- added R13: 100k, R3-LARGE_PADS, F.Cu at (123.2, 161.3)
- added R14: 100k, R3-LARGE_PADS, F.Cu at (139.7, 161.3)
- added R15: 100k, R3-LARGE_PADS, F.Cu at (156.2, 161.3)
- added R16: 100k, R3-LARGE_PADS, F.Cu at (172.7, 161.3)
- added R17: 100k, R3-LARGE_PADS, F.Cu at (189.2, 161.3)
- added R18: 100k, R3-LARGE_PADS, F.Cu at (205.7, 161.3)
- added R19: 100k, R3-LARGE_PADS, F.Cu at (222.2, 161.3)
- added R2: 10k, R3-LARGE_PADS, F.Cu at (141.6, 187.3)
- added R3: 10k, R3-LARGE_PADS, F.Cu at (144.8, 187.3)
- added R4: 1k, R3-LARGE_PADS, F.Cu at (100.3, 162.6)
- added R5: 1k, R3-LARGE_PADS, F.Cu at (116.8, 162.6)
- added R6: 1k, R3-LARGE_PADS, F.Cu at (133.3, 162.6)
- added R7: 1k, R3-LARGE_PADS, F.Cu at (149.9, 162.6)
- added R8: 1k, R3-LARGE_PADS, F.Cu at (166.4, 162.6)
- added R9: 1k, R3-LARGE_PADS, F.Cu at (182.9, 162.6)
- added Ref**: Val**, pad, F.Cu at (89.5, 116.2)
- added Ref**: Val**, pad, F.Cu at (230.5, 170.2)
- added Ref**: Val**, pad, F.Cu at (89.5, 196.2)
- added Ref**: Val**, pad, F.Cu at (230.5, 116.2)
- added Ref**: Val**, pad, F.Cu at (89.5, 170.2)
- added Ref**: Val**, pad, F.Cu at (230.5, 196.2)
- added U1: PCF8574, DIP-16__300_ELL, F.Cu at (158.1, 187.3)
Routing:
- net +5VD: track 0.00 -> 369.6 mm
- net DGND: track 0.00 -> 290.7 mm
- net +5V: track 0.00 -> 220.4 mm
- net GND: track 0.00 -> 132.7 mm
- net N-0000036: track 0.00 -> 83.0 mm
- net N-0000035: track 0.00 -> 82.2 mm
- net N-0000024: track 0.00 -> 67.0 mm
- net N-0000018: track 0.00 -> 60.5 mm
- net N-0000023: track 0.00 -> 49.4 mm
- net N-0000019: track 0.00 -> 40.6 mm
- net N-0000017: track 0.00 -> 36.1 mm
- net N-0000022: track 0.00 -> 26.9 mm
- net N-0000071: track 0.00 -> 24.8 mm
- net N-0000069: track 0.00 -> 24.1 mm
- net N-0000070: track 0.00 -> 23.3 mm
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- added copper zone on B.Cu, net DGND
- added copper zone on B.Cu, net GND
Other:
- board outline added: 149.9 x 88.9 mm
- net class Default: clearance 0.254 -> 0.25; trace_width 0.254 -> 0.508
- rule trace_clearance: 0.254 -> 0.25
- board text added: "2"
- board text added: "2xI C (5V-SCL-SDA-GND)"
- board text added: "A2-A1-A0"
- board text added: "SIMPLE RelayBoard v1.0"
